Commit message: wokring delta arm visual node/untested server ocde

File: workspace/src/percy_model/urdf/percy_model.gazebo.xacro (robot description, xacro)
@@ -55,7 +55,7 @@
 </plugin> -->
 </gazebo>
-    <gazebo reference="camera_link">
-    <material>Gazebo/Black</material>
-  <sensor type="camera" name="camera1">
+    <gazebo reference="camera_front_link">
+    <material>Gazebo/Blue</material>
+  <sensor type="camera" name="camera_front">
     <update_rate> 30.0 </update_rate>
     <camera name="head">
@@ -82,8 +82,88 @@
         <alwaysOn>true</alwaysOn>
         <updateRate>0.0</updateRate>
-        <cameraName>percy/camera1</cameraName>
+        <cameraName>percy/camera_front</cameraName>
         <imageTopicName>image_raw</imageTopicName>
         <cameraInfoTopicName>camera_info</cameraInfoTopicName>
-        <frameName>camera_link</frameName>
+        <frameName>camera_front_link</frameName>
+        <hackBaseline>0.07</hackBaseline>
+        <distortionK1>0.0</distortionK1>
+        <distortionK2>0.0</distortionK2>
+        <distortionK3>0.0</distortionK3>
+        <distortionT1>0.0</distortionT1>
+        <distortionT2>0.0</distortionT2>
+      </plugin>
+  </sensor>
+</gazebo>
+<gazebo reference="camera_rear_link">
+    <material>Gazebo/Red</material>
+  <sensor type="camera" name="camera_rear">
+    <update_rate> 30.0 </update_rate>
+    <camera name="rear">
+    <horizontal_fov>1.3962634</horizontal_fov>
+        <image>
+          <width>800</width>
+          <height>800</height>
+          <format>R8G8B8</format>
+        </image>
+        <clip>
+          <near>0.02</near>
+          <far>300</far>
+        </clip>
+        <noise>
+          <type>gaussian</type>
+          <!-- Noise is sampled independently per pixel on each frame.
+               That pixel's noise value is added to each of its color
+               channels, which at that point lie in the range [0,1]. -->
+          <mean>0.0</mean>
+          <stddev>0.007</stddev>
+        </noise>
+    </camera>
+    <plugin name="camera_controller" filename="libgazebo_ros_camera.so">
+        <alwaysOn>true</alwaysOn>
+        <updateRate>0.0</updateRate>
+        <cameraName>percy/camera_rear</cameraName>
+        <imageTopicName>image_raw</imageTopicName>
+        <cameraInfoTopicName>camera_info</cameraInfoTopicName>
+        <frameName>camera_rear_link</frameName>
+        <hackBaseline>0.07</hackBaseline>
+        <distortionK1>0.0</distortionK1>
+        <distortionK2>0.0</distortionK2>
+        <distortionK3>0.0</distortionK3>
+        <distortionT1>0.0</distortionT1>
+        <distortionT2>0.0</distortionT2>
+      </plugin>
+  </sensor>
+</gazebo>
+   <gazebo reference="camera_side_link">
+    <material>Gazebo/Black</material>
+  <sensor type="camera" name="camera_side">
+    <update_rate> 30.0 </update_rate>
+    <camera name="side">
+    <horizontal_fov>1.3962634</horizontal_fov>
+        <image>
+          <width>800</width>
+          <height>800</height>
+          <format>R8G8B8</format>
+        </image>
+        <clip>
+          <near>0.02</near>
+          <far>300</far>
+        </clip>
+        <noise>
+          <type>gaussian</type>
+          <!-- Noise is sampled independently per pixel on each frame.
+               That pixel's noise value is added to each of its color
+               channels, which at that point lie in the range [0,1]. -->
+          <mean>0.0</mean>
+          <stddev>0.007</stddev>
+        </noise>
+    </camera>
+    <plugin name="camera_controller" filename="libgazebo_ros_camera.so">
+        <alwaysOn>true</alwaysOn>
+        <updateRate>0.0</updateRate>
+        <cameraName>percy/camera_side</cameraName>
+        <imageTopicName>image_raw</imageTopicName>
+        <cameraInfoTopicName>camera_side_info</cameraInfoTopicName>
+        <frameName>camera_side_link</frameName>
         <hackBaseline>0.07</hackBaseline>
         <distortionK1>0.0</distortionK1>

File: workspace/src/percy_model/urdf/percy_model_v2.xacro (robot description, xacro)
@@ -589,5 +589,5 @@
         <origin xyz="0 0 ${body_height/2}"/>
 </joint>
-<link name="camera_link">
+<link name="camera_front_link">
     <collision>
         <geometry>
@@ -601,8 +601,44 @@
     </visual>
 </link>
-<joint name="camera_joint" type="fixed">
+<joint name="camera_front_joint" type="fixed">
     <axis xyz="0.0 1.0 0.0"/>
-    <origin xyz="${body_length/2} 0.0 ${-body_height/2 + (camera_link_height/2)+(link_width/2)}" rpy="0.0 0.75 0.0"/>
-        <child link="camera_link"/>
+    <origin xyz="${body_length/2} 0.0 ${-7*body_height/10}" rpy="0.0 0.9 0.0"/>
+        <child link="camera_front_link"/>
+        <parent link="origin"/>
+</joint>
+<link name="camera_side_link">
+    <collision>
+        <geometry>
+            <box size="${camera_link_width} ${camera_link_length} ${camera_link_height}"/>
+        </geometry>
+    </collision>
+    <visual>
+    <geometry>
+            <box size="${camera_link_width} ${camera_link_length} ${camera_link_height}"/>
+        </geometry>
+    </visual>
+</link>
+<joint name="camera_side_joint" type="fixed">
+    <axis xyz="0.0 1.0 0.0"/>
+    <origin xyz="0.0 ${body_width/2} ${-body_height-0.25}" rpy="0 0 -1.56"/>
+        <child link="camera_side_link"/>
+        <parent link="origin"/>
+    </joint>
+<link name="camera_rear_link">
+    <collision>
+        <geometry>
+            <box size="${camera_link_width} ${camera_link_length} ${camera_link_height}"/>
+        </geometry>
+    </collision>
+    <visual>
+    <geometry>
+            <box size="${camera_link_width} ${camera_link_length} ${camera_link_height}"/>
+        </geometry>
+    </visual>
+</link>
+<joint name="camera_rear_joint" type="fixed">
+    <axis xyz="0.0 1.0 0.0"/>
+    <origin xyz="${-1*body_length/2} 0.0 ${-body_height/2 + (camera_link_height/2)+(link_width/2)}" rpy="0.0 0.75 0.0"/>
+        <child link="camera_rear_link"/>
         <parent link="origin"/>
 </joint>
